Commit message: Add service /set_joint_angles and integrate plugin

File: xarm_description/urdf/common/common.gazebo.xacro (robot description, xacro)
@@ -19,4 +19,10 @@
         </xacro:if>
       </plugin>
+        <plugin name="set_initial_joint_angles_plugin" filename="libSetInitialJointAnglesPlugin.so">
+          <initial_joint_angles>
+            <joint name="joint6" angle="2.0" />
+            <joint name="joint4" angle="1.5" />
+          </initial_joint_angles>
+        </plugin>
     </gazebo>
   </xacro:macro>

Commit message: Add all joint to vel controller

File: xarm_description/urdf/common/common.gazebo.xacro (robot description, xacro)
@@ -20,8 +20,4 @@
       </plugin>
         <plugin name="set_initial_joint_angles_plugin" filename="libSetInitialJointAnglesPlugin.so">
-          <initial_joint_angles>
-            <joint name="joint6" angle="2.0" />
-            <joint name="joint4" angle="1.5" />
-          </initial_joint_angles>
         </plugin>
     </gazebo>
